File: kvm_switch/kvm_switch.kicad_sch (KiCad schematic)
At the start: 16 parts, among them J1 Conn_01x04_Pin, J2 Conn_01x06_Pin, J3 Conn_02x05_Odd_Even, U1 PC817, U2 PC817, U3 PC817

Commit message: 수정
Signed-off-by: Ju, Gyeong-min <jcmh74@gmail.com>
Parts:
- added J4: Conn_01x06_Pin, Connector_Molex:Molex_PicoBlade_53047-0610_1x06_P1.25mm_Vertical, symbol Connector:Conn_01x06_Pin
- added J5: Conn_02x05_Odd_Even, Connector_PinSocket_2.54mm:PinSocket_2x05_P2.54mm_Vertical, symbol Connector_Generic:Conn_02x05_Odd_Even
Connections:
- net ATX_PWRLED+: now also J4.6 (Pin_6), J5.2 (Pin_2)
- net ATX_PWRSW_A: now also J4.1 (Pin_1), J5.6 (Pin_6)
- net ATX_RSTSW_A: now also J4.3 (Pin_3), J5.7 (Pin_7)
- net GND2 renamed ATX_PWRLED-
- net ATX_PWRLED-: now also J4.2 (Pin_2), J4.4 (Pin_4), J4.5 (Pin_5), J5.5 (Pin_5), J5.8 (Pin_8)
- no-connect marks 5 -> 10
Other:
- moved on the sheet: J2, J3
