File: kvm_switch/kvm_switch.kicad_sch (KiCad schematic)
At the start: 18 parts, among them J1 Conn_01x04_Pin, J2 Conn_01x06_Pin, J3 Conn_02x05_Odd_Even, J4 Conn_01x06_Pin, J5 Conn_02x05_Odd_Even, U1 PC817, U2 PC817, U3 PC817

Commit message: 1차 주문 본
Signed-off-by: Ju, Gyeong-min <jcmh74@gmail.com>
Connections:
- net ATX_PWRLED-: now also J5.4 (Pin_4); no longer J2.5 (Pin_5), J3.8 (Pin_8), J4.2 (Pin_2), J5.8 (Pin_8), R3.2
- new net ATX_PWRSW_B: J2.5 (Pin_5), J3.8 (Pin_8), J4.2 (Pin_2), J5.8 (Pin_8), R3.2
- no-connect marks 10 -> 9
Other:
- company: (none) -> Amos Home
- title: (none) -> kvm_switch
- moved on the sheet: J1, J2, J3, J4, J5, R1, R10, R2, R3, R4, R5, R6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
