File: kvm_switch/kvm_switch.kicad_sch (KiCad schematic)
At the start: 18 parts, among them J1 Conn_01x04_Pin, J2 Conn_01x06_Pin, J3 Conn_02x05_Odd_Even, J4 Conn_01x06_Pin, J5 Conn_02x05_Odd_Even, U1 PC817, U2 PC817, U3 PC817

Commit message: PC817 패키지 타입을 SSO-4로 변경
Signed-off-by: Ju, Gyeong-min <jcmh74@gmail.com>
Parts:
- U1, U2, U3: footprint Package_SO:SOP-4_3.8x4.1mm_P2.54mm -> Package_SO:SSO-4_6.7x5.1mm_P2.54mm_Clearance8mm
