File: kvm_switch/kvm_switch.kicad_pcb (KiCad board)
At the start: 2 copper layers, 29 x 14.2 mm, 16 parts, among them J1 Conn_01x04_Pin, J2 Conn_01x06_Pin, J3 Conn_02x05_Odd_Even, U1 PC817, U2 PC817, U3 PC817

Commit message: 수정
Signed-off-by: Ju, Gyeong-min <jcmh74@gmail.com>
Parts:
- added J4: Conn_01x06_Pin, Connector_Molex:Molex_PicoBlade_53047-0610_1x06_P1.25mm_Vertical, F.Cu at (149.0, 83.8)
- added J5: Conn_02x05_Odd_Even, Connector_PinSocket_2.54mm:PinSocket_2x05_P2.54mm_Vertical, B.Cu at (156.0, 91.9)
- moved J3 0.70 mm to (145.7, 90.9)
Connections:
- net GND2 renamed /ATX_PWRLED-
Routing:
- net /ATX_PWRLED-: track 23.5 -> 54.8 mm
- net /ATX_RSTSW_A: track 9.15 -> 22.1 mm
- net /ATX_PWRSW_A: track 9.26 -> 21.7 mm
- net /ATX_PWRLED+: track 7.73 -> 19.4 mm
Other:
- board size 29 x 14.2 mm -> 40.5 x 14.2 mm
- board text added: "G"
- board text added: "L"
- board text added: "P"
- board text added: "P R G L"
- board text added: "PW+ PW- RS+ RS- LD- LD+"
- board text added: "R"

Commit message: 1차 주문 본
Signed-off-by: Ju, Gyeong-min <jcmh74@gmail.com>
Parts:
- moved J5 10.4 mm to (153.4, 81.8), turned to 180 degrees
Connections:
- J2 pad 5: /ATX_PWRLED- -> /ATX_PWRSW_B
- J3 pad 8: /ATX_PWRLED- -> /ATX_PWRSW_B
- J4 pad 2: /ATX_PWRLED- -> /ATX_PWRSW_B
- J5 pad 4: unconnected-(J5-Pin_4-Pad4) -> /ATX_PWRLED-
- J5 pad 8: /ATX_PWRLED- -> /ATX_PWRSW_B
- R3 pad 2: /ATX_PWRLED- -> /ATX_PWRSW_B
Routing:
- net /ATX_PWRSW_B: track 0.00 -> 22.9 mm
- net /ATX_PWRLED+: track 19.4 -> 31.8 mm
- net /ATX_PWRLED-: track 54.8 -> 45.7 mm
- net GND: track 16.3 -> 20.0 mm
- net /ATX_PWRSW_A: track 21.7 -> 24.2 mm
- net /ATX_RSTSW_A: track 22.1 -> 19.9 mm
Other:
- board size 40.5 x 14.2 mm -> 40.2 x 14.2 mm
- board text added: "NUC"
- board text added: "P R L"
- board text added: "X"
- board text removed: "P R G L"
